File: PCB/PCB.kicad_sch (KiCad schematic)
At the start: 0 parts

Commit message: added PCB designs
Parts:
- added U1: AS5600, symbol Components:AS5600
- added U2: A4988, symbol Components:A4988
- added U3: MP1584, symbol Components:MP1584

Commit message: Updated files
Parts:
- removed U1: AS5600, symbol Components:AS5600
- removed U2: A4988, symbol Components:A4988
- removed U3: MP1584, symbol Components:MP1584
- added U1: DC-DC Converter, Module:DC-DC Converter, symbol Joint_Components:DC-DC_Converter
- added U2: A4988, symbol Joint_Components:A4988
- added U3: AS5600, symbol Joint_Components:AS5600
- added U4: ESP32-C3 Super Mini, symbol Joint_Components:ESP32-C3_Super_Mini
Connections:
- new net: U3.1 (VCC), U3.7 (GPO), U4.6 (3v3)
- new net: U1.5 (OUT-), U2.9 (GND), U3.2 (GND), U4.8 (GND)
- new net: U3.3 (OUT), U4.3 (A0)
- new net: U2.1 (EN), U4.12 (SCK)
- new net: U1.8 (OUT+), U2.10 (VDD), U2.2 (MS1), U2.3 (MS2), U2.4 (MS3), U4.7 (5v)
- new net: U2.5 (RST), U2.6 (SLP)
- new net: U2.7 (DIR), U4.14 (MOSI)
- new net: U2.8 (STEP), U4.13 (MISO)
- new net +12V: U1.4 (IN+), U2.16 (VMOT)
- new net GND: U1.1 (IN-), U2.15 (GND)
- no-connect marks 0 -> 7
